File: Hardware/PCB/smart home/smart home.kicad_sch (KiCad schematic)
At the start: 51 parts, among them M1 Fan, Q1 BC547C, Q2 BC547C, Q3 BC547, Q6 BC547C, Q7 BC547C, Q8 BC547C, Q9 BC547C, SW1 SW_SPST, SW2 SW_SPST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

Commit message: Unscrew folder structure, add updated gerbers
Parts:
- removed Pot1, Pot2, Pot3, Pot4: ~, symbol smarthome:Pot
- removed R21, R22: 100k, symbol Device:R
- removed SW3, SW7: SW_SPST, symbol Switch:SW_SPST
- removed SW6: SW_Push, symbol Switch:SW_Push
- added C1: 4.7µF, Library:CAPPRD200W45D500H500, symbol Device:C_Polarized
- added H1, H2, H3, H4: MountingHole, MountingHole:MountingHole_2.2mm_M2, symbol Mechanical:MountingHole
- added RV1, RV3B1, RV3G1, RV3R1: 10k, Connector_PinHeader_2.54mm:PinHeader_1x03_P2.54mm_Vertical, symbol Device:R_Potentiometer
- added SW6, SW9: SW_SPST, Connector_PinHeader_2.54mm:PinHeader_1x02_P2.54mm_Vertical, symbol Switch:SW_SPST
- added SW7: SW_Push, Connector_PinHeader_2.54mm:PinHeader_1x02_P2.54mm_Vertical, symbol Switch:SW_Push
- BT1, M1, SW1, SW2, SW4, SW5: footprint (none) -> Connector_PinHeader_2.54mm:PinHeader_1x02_P2.54mm_Vertical
- HC–SR505PIR1: footprint (none) -> Connector_PinHeader_2.54mm:PinHeader_1x03_P2.54mm_Vertical
- LCD_20x1: footprint (none) -> Connector_PinHeader_2.54mm:PinHeader_1x04_P2.54mm_Vertical
- Q1, Q2, Q3, Q6, Q7, Q8, Q9: footprint Package_TO_SOT_THT:TO-92_Inline -> Package_TO_SOT_THT:TO-92_HandSolder
- R1, R10, R11, R12, R13, R14, R15, R16, R17, R18, R19, R2, R24, R3, R4, R5, R6, R7, R8, R9: footprint (none) -> Resistor_THT:R_Axial_DIN0207_L6.3mm_D2.5mm_P10.16mm_Horizontal
- R20: value 100k -> 10k; footprint (none) -> Resistor_THT:R_Axial_DIN0207_L6.3mm_D2.5mm_P10.16mm_Horizontal
- R23: footprint OptoDevice:R_LDR_10x8.5mm_P7.6mm_Vertical -> Connector_PinHeader_2.54mm:PinHeader_1x02_P2.54mm_Vertical
- RGB1, RGB2, RGB3, RGB4: footprint (none) -> Connector_PinSocket_2.54mm:PinSocket_2x02_P2.54mm_Vertical
Connections:
- net Fan switch is gone; now on net R2_S2: SW2.2 (B)
- net MC_enable is gone; now on net +9V: HC–SR505PIR1.3 (Possitive_ps)
- net R5B enable is gone; now on net R3B enable: R14.2
- net fan enanble is gone; now on net fan enable: A1.14 (D11)
- net +5V: now also LCD_20x1.3 (Vcc), RV1.3, RV3B1.3, RV3G1.3, RV3R1.3; no longer SW1.1 (A), SW2.1 (A), SW4.1, SW5.1
- net C_button_1: now also SW5.2; no longer R20.1, SW4.2
- net C_button_2: now also SW4.2; no longer SW5.2
- net C_button_3: now also SW7.2
- net GND: now also SW1.1 (A), SW2.1 (A), SW4.1, SW5.1, C1.2, RV1.1, RV3B1.1, RV3G1.1, RV3R1.1, SW6.1 (A), SW7.1, SW9.1 (A)
- net LDR: now also R20.1
- net MC_signal: no longer A1.16 (D13)
- net R1-D: now also RV1.2
- net R3-B: now also RV3B1.2
- net R3-G: now also RV3G1.2
- net R3-R: now also RV3R1.2
- net R3_S1: now also SW9.2 (B)
- net VCC: now also C1.1; no longer LCD_20x1.3 (Vcc)
- new net fan switch: A1.16 (D13), SW6.2 (B)
Other:
- note added: "Mounting holes"
- moved on the sheet: R23
