File: Hardware/PCB/smart home/smart home.kicad_pcb (KiCad board)
At the start: 2 copper layers, 103 x 93 mm, 54 parts, among them M1 Fan, Q1 BC547C, Q2 BC547C, Q3 BC547, Q6 BC547C, Q7 BC547C, Q8 BC547C, Q9 BC547C, SW1 SW_SPST, SW2 SW_SPST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

Commit message: update kicad proj to current. new pcb, gerber, etc.
Signed-off-by: bobo <usnameos@outlook.com>
Parts:
- moved R20 14.3 mm to (115.1, 45.5), turned to 180 degrees
- moved LCD_20x1 7.03 mm to (106.0, 62.5)
- moved R23 7.02 mm to (108.3, 57.0)
- moved RV1 6.58 mm to (111.0, 80.5)
- moved RV3B1 6.58 mm to (111.1, 67.0)
- moved RV3G1 6.58 mm to (111.0, 71.5)
- moved RV3R1 6.58 mm to (111.0, 76.0)
- moved SW6 6.58 mm to (108.8, 85.0)
- moved SW9 6.55 mm to (108.3, 52.0)
- moved SW1 2.55 mm to (65.0, 78.5)
- moved SW4 2.55 mm to (64.7, 83.5)
- moved Q2 2.10 mm to (55.0, 50.0)
- moved R14 1.00 mm to (56.4, 89.5)
Routing:
- net GND: track 378.9 -> 10.9 mm, vias 0 -> 2
- net LDR: track 19.1 -> 29.9 mm
- net VCC: track 322.8 -> 327.4 mm
- net +5V: track 73.8 -> 77.9 mm
- net R3_S1: track 8.58 -> 12.1 mm
- net R2_S1: track 14.0 -> 17.3 mm
- net R1-D: track 14.0 -> 10.8 mm
- net C_button_2: track 15.2 -> 17.9 mm
- net SCL: track 13.5 -> 15.6 mm
- net Net-(Q2-B): track 7.69 -> 9.52 mm
- net R3-R: track 11.7 -> 10.0 mm
- net SDA: track 9.90 -> 11.1 mm
- net fan switch: track 11.5 -> 10.5 mm
- net R3-G: track 10.9 -> 9.88 mm
- net Net-(RGB4-G): track 7.63 -> 6.92 mm
